File: Eagle/EncoderShield/Encoder_Breakout.brd (EAGLE design)
At the start: 100 x 80 mm, 32 parts, among them IC1 MC33932, IC2 74LVC1G04DCK, IC3 74LVC1G04DCK, IC4 7806DT

Commit message: Add files via upload
Parts:
- removed C1, C2: (no value), rcl:153CLV-0810
- removed C3: (no value), rcl:153CLV-0405
- removed CCPA_C, CCPB_C, FBA_C, FBB_C: (no value), resistor:C0805
- removed ER1, ER2, FBA_PULLDWN, FBB_PULLDWN, PULLDWN_D1, PULLDWN_D3, PULLDWN_EN/!D2, PULLDWN_EN/!D4, PWRR, SFA_PULLUP, SFB_PULLUP: (no value), rcl:R0805
- removed ERROR1, ERROR2, POWER: (no value), eagle-ltspice:LED_1206
- removed IC1: MC33932, freescale:HSOP44
- removed IC2, IC3: 74LVC1G04DCK, 74xx-little-de:SC70-5
- removed IC4: 7806DT, linear:TO252
- removed U$3, U$4, U$5: TERM_QUICK, TERM_QUICK:TERM_QUICK
- added JP10, JP4, JP5, JP6, JP7, JP8, JP9: (no value), pinhead:1X04
- added SV1, SV2, SV3, SV4: (no value), con-lsta:FE06
- added SV10, SV11, SV12, SV7, SV8, SV9: (no value), con-lstb:MA03-1
- added SV5, SV6: (no value), con-lsta:FE05-1
- added U$1: TAG, TAG:TAG
- JP3: device pinhead:1X02 -> pinhead:1X04
- moved JP3 122.6 mm to (47.0, 36.8), turned to 270 degrees
- moved JP2 113.6 mm to (55.9, 17.8), turned to 270 degrees
- moved JP1 103.2 mm to (55.9, 36.8), turned to 270 degrees
Connections:
- removed net !SFA: IC1.44, IC2.2, SFA_PULLUP.2
- removed net !SFB: IC1.22, IC3.2, SFB_PULLUP.2
- removed net CCPA: CCPA_C.2, IC1.41
- removed net CCPB: CCPB_C.2, IC1.19
- removed net D1: IC1.1, PULLDWN_D1.2
- removed net D3: IC1.23, PULLDWN_D3.2
- removed net EN/!D2: IC1.3, PULLDWN_EN/!D2.2
- removed net EN/!D4: IC1.25, PULLDWN_EN/!D4.2
- removed net FBA: FBA_C.1, FBA_PULLDWN.2, IC1.2
- removed net FBB: FBB_C.1, FBB_PULLDWN.2, IC1.24
- removed net IN1: IC1.43
- removed net IN2: IC1.42
- removed net IN3: IC1.21
- removed net IN4: IC1.20
- removed net N$1: ER2.1, IC3.4
- removed net N$15: ER1.2, ERROR1.A
- removed net N$16: ER2.2, ERROR2.A
- removed net N$3: POWER.A, PWRR.2
- removed net N$7: ER1.1, IC2.4
- removed net OUT1: IC1.7, IC1.8, IC1.9, U$3.P$1
- removed net OUT2: IC1.36, IC1.37, IC1.38, U$3.P$2
- removed net OUT3: IC1.29, IC1.30, IC1.31, U$4.P$1
- removed net OUT4: IC1.14, IC1.15, IC1.16, U$4.P$2
- removed net VPWR: C1.+, C2.+, CCPA_C.1, CCPB_C.1, IC1.17, IC1.18, IC1.26, IC1.27, IC1.28, IC1.39, IC1.4, IC1.40, IC1.5, IC1.6, IC4.1, JP3.1, U$5.P$1
- new net ENA1: B1.34, SV5.5
- new net ENA2: B1.36, SV6.5
- new net ENC3_A: B1.18, JP3.3
- new net ENC3_B: B1.26, JP3.4
- new net ENC4_A: B1.19, JP4.3
- new net ENC4_B: B1.28, JP4.4
- new net ENC5_A: B1.20, JP5.3
- new net ENC5_B: B1.30, JP5.4
- new net ENC6_A: B1.21, JP6.3
- new net ENC6_B: B1.32, JP6.4
- new net MISO: B1.50, SV1.3, SV2.3, SV3.3, SV4.3
- new net MOSI: B1.51, SV1.4, SV2.4, SV3.4, SV4.4
- new net PWM1: B1.4, SV7.3
- new net PWM10: B1.13, SV6.4
- new net PWM2: B1.5, SV8.3
- new net PWM3: B1.6, SV9.3
- new net PWM4: B1.7, SV10.3
- new net PWM5: B1.8, SV11.3
- new net PWM6: B1.9, SV12.3
- new net PWM7: B1.10, SV5.3
- new net PWM8: B1.11, SV5.4
- new net PWM9: B1.12, SV6.3
- new net SCK: B1.52, SV1.5, SV2.5, SV3.5, SV4.5
- new net SCL: B1.SCL, JP10.3, JP7.3, JP8.3, JP9.3
- new net SDA: B1.SDA, JP10.4, JP7.4, JP8.4, JP9.4
- new net SS: B1.53
- new net SS1: B1.38, SV1.6
- new net SS2: B1.40, SV2.6
- new net SS3: B1.42, SV3.6
- new net SS4: B1.44, SV4.6
- net 5V_PWR: now also B1.5V, B1.5V@1, B1.5V@2, JP10.1, JP3.1, JP4.1, JP5.1, JP6.1, JP7.1, JP8.1, JP9.1, SV1.1, SV10.2, SV11.2, SV12.2, SV2.1, SV3.1, SV4.1, SV5.1, SV6.1, SV7.2, SV8.2, SV9.2; no longer C3.+, IC2.5, IC3.5, IC4.2, PWRR.1, SFA_PULLUP.1, SFB_PULLUP.1
- net ENC1_A: now also B1.2
- net ENC1_B: now also B1.22
- net ENC2_A: now also B1.3
- net ENC2_B: now also B1.24
- net GND: now also B1.GND, B1.GND@1, B1.GND@2, B1.GND@3, B1.GND@4, JP10.2, JP4.2, JP5.2, JP6.2, JP7.2, JP8.2, JP9.2, SV1.2, SV10.1, SV11.1, SV12.1, SV2.2, SV3.2, SV4.2, SV5.2, SV6.2, SV7.1, SV8.1, SV9.1; no longer C1.-, C2.-, C3.-, ERROR1.C, ERROR2.C, FBA_C.2, FBA_PULLDWN.1, FBB_C.2, FBB_PULLDWN.1, IC1.10, IC1.11, IC1.12, IC1.13, IC1.32, IC1.33, IC1.34, IC1.35, IC1.EH@1, IC1.EH@2, IC1.EH@3, IC2.3, IC3.3, IC4.3, POWER.C, PULLDWN_D1.1, PULLDWN_D3.1, PULLDWN_EN/!D2.1, PULLDWN_EN/!D4.1, U$5.P$2
Routing:
- net 5V_PWR: track 0.00 -> 243.0 mm
- net ENA1: track 0.00 -> 88.3 mm
- net ENA2: track 0.00 -> 84.2 mm
- net ENC4_B: track 0.00 -> 70.5 mm, vias 0 -> 1
- net ENC6_A: track 0.00 -> 68.2 mm
- net ENC6_B: track 0.00 -> 66.1 mm
- net ENC5_B: track 0.00 -> 59.9 mm
- net PWM4: track 0.00 -> 59.1 mm
- net ENC5_A: track 0.00 -> 55.0 mm, vias 0 -> 1
- net ENC2_B: track 0.00 -> 53.7 mm
- net ENC3_B: track 0.00 -> 53.6 mm
- net ENC4_A: track 0.00 -> 52.1 mm, vias 0 -> 1
- net PWM10: track 0.00 -> 51.2 mm
- net MOSI: track 0.00 -> 49.7 mm
- net PWM9: track 0.00 -> 46.7 mm
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- added copper zone on layer 1, net GND
- added copper zone on layer 16, net GND
Other:
- board size 100 x 80 mm -> 100 x 53.3 mm
- board text added: "(10)"
- board text added: "(11)"
- board text added: "(12)"
- board text added: "(13)"
- board text added: "(18)"
- board text added: "(19)"
- board text added: "(20)"
- board text added: "(21)"
- board text added: "(26)"
- board text added: "(28)"
- board text added: "(30)"
- board text added: "(32)"
- board text added: "(34)"
- board text added: "(36)"
- board text added: "(38)"
- board text added: "(4)"
- board text added: "(40)"
- board text added: "(42)"
- board text added: "(44)"
- board text added: "(5)"
- board text added: "(6)"
- board text added: "(7)"
- board text added: "(8)"
- board text added: "(9)"
- board text added: "01-2019"
- board text added: "2xPWM/ENA"
- board text added: "5V"
- board text added: "A(2)"
- board text added: "A(3)"
- board text added: "Arduino Mega Robot Interface"
- board text added: "B(22)"
- board text added: "B(24)"
- board text added: "Brayden DeBoon"
- board text added: "ENCODERS"
- board text added: "GND"
- board text added: "I2C"
- board text added: "MISO"
- board text added: "MOSI"
- board text added: "PWM"
- board text added: "SCK"
- board text added: "SCL"
- board text added: "SDA"
- board text added: "SPI"
- board text added: "SS"
