File: Eagle/EncoderShield/Encoder_Breakout.sch (EAGLE design)
At the start: 32 parts, among them IC1 MC33932, IC2 74LVC1G04DCK, IC3 74LVC1G04DCK, IC4 7806DT

Commit message: Add files via upload
Parts:
- removed C1, C2: (no value), rcl:CPOL-US153CLV-0810
- removed C3: (no value), rcl:CPOL-EU153CLV-0405
- removed CCPA_C, CCPB_C, FBA_C, FBB_C: (no value), resistor:C-USC0805
- removed ER1, ER2, FBA_PULLDWN, FBB_PULLDWN, PULLDWN_D1, PULLDWN_D3, PULLDWN_EN/!D2, PULLDWN_EN/!D4, PWRR, SFA_PULLUP, SFB_PULLUP: (no value), rcl:R-US_R0805
- removed ERROR1, ERROR2, POWER: (no value), eagle-ltspice:LED_E
- removed IC1: MC33932, freescale:MC33932
- removed IC2, IC3: 74LVC1G04DCK, 74xx-little-de:74LVC1G04DCK
- removed IC4: 7806DT, linear:7806DT
- removed U$3, U$4, U$5: TERM_QUICK, TERM_QUICK:TERM_QUICK
- added JP10, JP4, JP5, JP6, JP7, JP8, JP9: (no value), pinhead:PINHD-1X4
- added SV1, SV2, SV3, SV4: (no value), con-lsta:FE06-1
- added SV10, SV11, SV12, SV7, SV8, SV9: (no value), con-lstb:MA03-1
- added SV5, SV6: (no value), con-lsta:FE05-1
- added U$1: TAG, TAG:TAG
- JP3: device pinhead:PINHD-1X2 -> pinhead:PINHD-1X4
Connections:
- removed net !SFA: IC1.!SFA, IC2A.I, SFA_PULLUP.2
- removed net !SFB: IC1.!SFB, IC3A.I, SFB_PULLUP.2
- removed net CCPA: CCPA_C.2, IC1.CCPA
- removed net CCPB: CCPB_C.2, IC1.CCPB
- removed net D1: IC1.D1, PULLDWN_D1.2
- removed net D3: IC1.D3, PULLDWN_D3.2
- removed net EN/!D2: IC1.EN/!D2, PULLDWN_EN/!D2.2
- removed net EN/!D4: IC1.EN/!D4, PULLDWN_EN/!D4.2
- removed net FBA: FBA_C.1, FBA_PULLDWN.2, IC1.FBA
- removed net FBB: FBB_C.1, FBB_PULLDWN.2, IC1.FBB
- removed net IN1: IC1.IN1
- removed net IN2: IC1.IN2
- removed net IN3: IC1.IN3
- removed net IN4: IC1.IN4
- removed net N$1: ER2.1, IC3A.O
- removed net N$15: ER1.2, ERROR1.A
- removed net N$16: ER2.2, ERROR2.A
- removed net N$3: POWER.A, PWRR.2
- removed net N$7: ER1.1, IC2A.O
- removed net OUT1: IC1.OUT1, IC1.OUT1@1, IC1.OUT1@2, U$3.P$1
- removed net OUT2: IC1.OUT2, IC1.OUT2@1, IC1.OUT2@2, U$3.P$2
- removed net OUT3: IC1.OUT3, IC1.OUT3@1, IC1.OUT3@2, U$4.P$1
- removed net OUT4: IC1.OUT4, IC1.OUT4@1, IC1.OUT4@2, U$4.P$2
- removed net VPWR: C1.+, C2.+, CCPA_C.1, CCPB_C.1, IC1.VPWRA, IC1.VPWRA@1, IC1.VPWRA@2, IC1.VPWRA@3, IC1.VPWRA@4, IC1.VPWRB, IC1.VPWRB@1, IC1.VPWRB@2, IC1.VPWRB@3, IC1.VPWRB@4, IC4.VI, JP3.1, U$5.P$1
- new net ENA1: B1.34, SV5.5
- new net ENA2: B1.36, SV6.5
- new net ENC3_A: B1.18(TX1), JP3.3
- new net ENC3_B: B1.26, JP3.4
- new net ENC4_A: B1.19(RX1), JP4.3
- new net ENC4_B: B1.28, JP4.4
- new net ENC5_A: B1.20(SDA), JP5.3
- new net ENC5_B: B1.30, JP5.4
- new net ENC6_A: B1.21(SCL), JP6.3
- new net ENC6_B: B1.32, JP6.4
- new net MISO: B1.50/MISO, SV1.3, SV2.3, SV3.3, SV4.3
- new net MOSI: B1.51/MOSI, SV1.4, SV2.4, SV3.4, SV4.4
- new net PWM1: B1.4, SV7.3
- new net PWM10: B1.13, SV6.4
- new net PWM2: B1.5, SV8.3
- new net PWM3: B1.6, SV9.3
- new net PWM4: B1.7, SV10.3
- new net PWM5: B1.8, SV11.3
- new net PWM6: B1.9, SV12.3
- new net PWM7: B1.10, SV5.3
- new net PWM8: B1.11, SV5.4
- new net PWM9: B1.12, SV6.3
- new net SCK: B1.52/SCK, SV1.5, SV2.5, SV3.5, SV4.5
- new net SCL: B1.SCL, JP10.3, JP7.3, JP8.3, JP9.3
- new net SDA: B1.SDA, JP10.4, JP7.4, JP8.4, JP9.4
- new net SS: B1.53/!CS
- new net SS1: B1.38, SV1.6
- new net SS2: B1.40, SV2.6
- new net SS3: B1.42, SV3.6
- new net SS4: B1.44, SV4.6
- net 5V_PWR: now also B1.5V, JP10.1, JP3.1, JP4.1, JP5.1, JP6.1, JP7.1, JP8.1, JP9.1, SV1.1, SV10.2, SV11.2, SV12.2, SV2.1, SV3.1, SV4.1, SV5.1, SV6.1, SV7.2, SV8.2, SV9.2; no longer C3.+, IC2P.VCC, IC3P.VCC, IC4.VO, PWRR.1, SFA_PULLUP.1, SFB_PULLUP.1
- net ENC1_A: now also B1.2
- net ENC1_B: now also B1.22
- net ENC2_A: now also B1.3
- net ENC2_B: now also B1.24
- net GND: now also B1.GND, B1.GND@2, B1.GND@3, JP10.2, JP4.2, JP5.2, JP6.2, JP7.2, JP8.2, JP9.2, SV1.2, SV10.1, SV11.1, SV12.1, SV2.2, SV3.2, SV4.2, SV5.2, SV6.2, SV7.1, SV8.1, SV9.1; no longer C1.-, C2.-, C3.-, ERROR1.C, ERROR2.C, FBA_C.2, FBA_PULLDWN.1, FBB_C.2, FBB_PULLDWN.1, IC1.EH@1, IC1.EH@2, IC1.EH@3, IC1.PGNDA, IC1.PGNDA@1, IC1.PGNDA@2, IC1.PGNDA@3, IC1.PGNDB, IC1.PGNDB@1, IC1.PGNDB@2, IC1.PGNDB@3, IC2P.GND, IC3P.GND, IC4.GND, POWER.C, PULLDWN_D1.1, PULLDWN_D3.1, PULLDWN_EN/!D2.1, PULLDWN_EN/!D4.1, U$5.P$2
