File: Eagle/LocMap/LocationMapper.sch (EAGLE design)
At the start: 44 parts, among them Q1 8/16/20MHz, U1 ATMEGA328

Commit message: Add files via upload
Parts:
- added R17, R18: (no value), resistor:R-US_R0805
- added U$17, U$18: LED_LM, LED_LM:LED_LM
Connections:
- new net N$22: R18.1, U$18.P$1
- new net N$27: R17.1, U$17.P$1
- net GND: now also R17.2, R18.2
- net N$1: now also U$6.P$1; no longer U$1.P$2
- net N$10: now also U$5.P$1; no longer U$9.P$2
- net N$2: now also U$7.P$1; no longer U$2.P$2
- net N$3: now also U$8.P$1; no longer U$3.P$2
- net N$4: now also U$9.P$1; no longer U$4.P$2
- net N$5: now also U$10.P$1; no longer U$5.P$2
- net N$6: now also U$1.P$1; no longer U$10.P$2
- net N$7: now also U$2.P$1; no longer U$6.P$2
- net N$8: now also U$3.P$1; no longer U$7.P$2
- net N$9: now also U$4.P$1; no longer U$8.P$2
- net VDD: now also U$1.P$2, U$10.P$2, U$17.P$2, U$18.P$2, U$2.P$2, U$3.P$2, U$4.P$2, U$5.P$2, U$6.P$2, U$7.P$2, U$8.P$2, U$9.P$2; no longer U$1.P$1, U$10.P$1, U$2.P$1, U$3.P$1, U$4.P$1, U$5.P$1, U$6.P$1, U$7.P$1, U$8.P$1, U$9.P$1

Commit message: Add files via upload
Parts:
- added PAD3, PAD4, PAD5: (no value), wirepad:2,54/1,1
Connections:
- removed net RAW: PAD1.P
- net GND: now also PAD4.P, PAD5.P; no longer PAD2.P
- net RXI: now also PAD2.P
- net TXO: now also PAD1.P
- net VCC: now also PAD3.P
Other:
- moved on the sheet: PAD1, PAD2
Changed lines of the file:
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@@
 <?xml version="1.0" encoding="utf-8"?>
 <!DOCTYPE eagle SYSTEM "eagle.dtd">
-<eagle version="8.6.0">
+<eagle version="8.0.1">
 <drawing>
 <settings>
@@
 </variantdefs>
 <classes>
-<class number="0" name="default" width="0.2032" drill="0.1016">
+<class number="0" name="default" width="0.2032" drill="0.2032">
 <clearance class="0" value="0.2032"/>
 </class>
@@
 </classes>
 <parts>
-<part name="R1" library="resistor" library_urn="urn:adsk.eagle:library:348" deviceset="R-US_" device="R0805" package3d_urn="urn:adsk.eagle:package:26059/1"/>
-<part name="R2" library="resistor" library_urn="urn:adsk.eagle:library:348" deviceset="R-US_" device="R0805" package3d_urn="urn:adsk.eagle:package:26059/1"/>
-<part name="R3" library="resistor" library_urn="urn:adsk.eagle:library:348" deviceset="R-US_" device="R0805" package3d_urn="urn:adsk.eagle:package:26059/1"/>
-<part name="R4" library="resistor" library_urn="urn:adsk.eagle:library:348" deviceset="R-US_" device="R0805" package3d_urn="urn:adsk.eagle:package:26059/1"/>
-<part name="R5" library="resistor" library_urn="urn:adsk.eagle:library:348" deviceset="R-US_" device="R0805" package3d_urn="urn:adsk.eagle:package:26059/1"/>
-<part name="R6" library="resistor" library_urn="urn:adsk.eagle:library:348" deviceset="R-US_" device="R0805" package3d_urn="urn:adsk.eagle:package:26059/1"/>
-<part name="R7" library="resistor" library_urn="urn:adsk.eagle:library:348" deviceset="R-US_" device="R0805" package3d_urn="urn:adsk.eagle:package:26059/1"/>
-<part name="R8" library="resistor" library_urn="urn:adsk.eagle:library:348" deviceset="R-US_" device="R0805" package3d_urn="urn:adsk.eagle:package:26059/1"/>
-<part name="R9" library="resistor" library_urn="urn:adsk.eagle:library:348" deviceset="R-US_" device="R0805" package3d_urn="urn:adsk.eagle:package:26059/1"/>
-<part name="R10" library="resistor" library_urn="urn:adsk.eagle:library:348" deviceset="R-US_" device="R0805" package3d_urn="urn:adsk.eagle:package:26059/1"/>
+<part name="R1" library="resistor" deviceset="R-US_" device="R0805"/>
+<part name="R2" library="resistor" deviceset="R-US_" device="R0805"/>
+<part name="R3" library="resistor" deviceset="R-US_" device="R0805"/>
+<part name="R4" library="resistor" deviceset="R-US_" device="R0805"/>
+<part name="R5" library="resistor" deviceset="R-US_" device="R0805"/>
+<part name="R6" library="resistor" deviceset="R-US_" device="R0805"/>
+<part name="R7" library="resistor" deviceset="R-US_" device="R0805"/>
+<part name="R8" library="resistor" deviceset="R-US_" device="R0805"/>
+<part name="R9" library="resistor" deviceset="R-US_" device="R0805"/>
+<part name="R10" library="resistor" deviceset="R-US_" device="R0805"/>
 <part name="U$11" library="ULN2803A" deviceset="ULN2803A" device=""/>
 <part name="U$12" library="ULN2803A" deviceset="ULN2803A" device=""/>
-<part name="SUPPLY1" library="supply2" library_urn="urn:adsk.eagle:library:372" deviceset="GND" device=""/>
-<part name="SUPPLY2" library="supply2" library_urn="urn:adsk.eagle:library:372" deviceset="GND" device=""/>
+<part name="SUPPLY1" library="supply2" deviceset="GND" device=""/>
+<part name="SUPPLY2" library="supply2" deviceset="GND" device=""/>
 <part name="U$14" library="7SEG" deviceset="7SEG" device=""/>
 <part name="U$15" library="7SEG_DRIVER" deviceset="7SEG_DRIVER" device=""/>
-<part name="R11" library="resistor" library_urn="urn:adsk.eagle:library:348" deviceset="R-US_" device="R0805" package3d_urn="urn:adsk.eagle:package:26059/1"/>
+<part name="R11" library="resistor" deviceset="R-US_" device="R0805"/>
 <part name="U$13" library="7SEG" deviceset="7SEG" device=""/>
 <part name="U$16" library="7SEG_DRIVER" deviceset="7SEG_DRIVER" device=""/>
-<part name="R12" library="resistor" library_urn="urn:adsk.eagle:library:348" deviceset="R-US_" device="R0805" package3d_urn="urn:adsk.eagle:package:26059/1"/>
+<part name="R12" library="resistor" deviceset="R-US_" device="R0805"/>
 <part name="R13" library="SparkFun" deviceset="RESISTOR" device="0603-RES" value="10K"/>
 <part name="GND3" library="SparkFun" deviceset="GND" device=""/>
@@
 <part name="S1" library="Testing" deviceset="SWITCH-MOMENTARY-2" device="SMD-ALT01" value="Reset"/>
 <part name="Q1" library="Testing" deviceset="RESONATOR" device="1:1" value="8/16/20MHz"/>
-<part name="PAD1" library="wirepad" library_urn="urn:adsk.eagle:library:412" deviceset="2,54/1,1" device="" package3d_urn="urn:adsk.eagle:package:30836/1"/>
-<part name="PAD2" library="wirepad" library_urn="urn:adsk.eagle:library:412" deviceset="2,54/1,1" device="" package3d_urn="urn:adsk.eagle:package:30836/1"/>
+<part name="PAD1" library="wirepad" deviceset="2,54/1,1" device=""/>
+<part name="PAD2" library="wirepad" deviceset="2,54/1,1" device=""/>
 <part name="SJ2" library="SparkFun-Passives" deviceset="SOLDERJUMPER" device="NC" value=""/>
 <part name="SJ3" library="SparkFun-Passives" deviceset="SOLDERJUMPER" device="NC" value=""/>
@@
 <part name="U$10" library="LED_LM" deviceset="LED_LM" device=""/>
 <part name="U$17" library="LED_LM" deviceset="LED_LM" device=""/>
-<part name="R17" library="resistor" library_urn="urn:adsk.eagle:library:348" deviceset="R-US_" device="R0805" package3d_urn="urn:adsk.eagle:package:26059/1"/>
+<part name="R17" library="resistor" deviceset="R-US_" device="R0805"/>
 <part name="U$18" library="LED_LM" deviceset="LED_LM" device=""/>
-<part name="R18" library="resistor" library_urn="urn:adsk.eagle:library:348" deviceset="R-US_" device="R0805" package3d_urn="urn:adsk.eagle:package:26059/1"/>
+<part name="R18" library="resistor" deviceset="R-US_" device="R0805"/>
+<part name="PAD3" library="wirepad" deviceset="2,54/1,1" device=""/>
+<part name="PAD4" library="wirepad" deviceset="2,54/1,1" device=""/>
+<part name="PAD5" library="wirepad" deviceset="2,54/1,1" device=""/>
 </parts>
 <sheets>
@@
 <attribute name="VALUE" x="253.492" y="61.722" size="1.778" layer="96"/>
 </instance>
-<instance part="PAD1" gate="1" x="363.22" y="66.04" rot="R180"/>
-<instance part="PAD2" gate="1" x="363.22" y="58.42" rot="R180"/>
+<instance part="PAD1" gate="1" x="363.22" y="53.34" rot="R180"/>
+<instance part="PAD2" gate="1" x="363.22" y="45.72" rot="R180"/>
 <instance part="SJ2" gate="1" x="237.49" y="87.63" rot="R90"/>
 <instance part="SJ3" gate="1" x="228.6" y="81.28" rot="R180"/>
@@
 <instance part="U$18" gate="G$1" x="-60.96" y="68.58" rot="R180"/>
 <instance part="R18" gate="G$1" x="-50.8" y="55.88"/>
+<instance part="PAD3" gate="1" x="363.22" y="60.96" rot="R180"/>
+<instance part="PAD4" gate="1" x="363.22" y="68.58" rot="R180"/>
+<instance part="PAD5" gate="1" x="363.22" y="35.56" rot="R180"/>
 </instances>
 <busses>
@@
 </segment>
 <segment>
-<pinref part="PAD2" gate="1" pin="P"/>
-<wire x1="360.68" y1="58.42" x2="358.14" y2="58.42" width="0.1524" layer="91"/>
-<label x="358.14" y="58.42" size="1.778" layer="95" rot="R180" xref="yes"/>
-</segment>
-<segment>
 <wire x1="288.29" y1="118.11" x2="290.83" y2="118.11" width="0.1524" layer="91"/>
 <pinref part="JP1" gate="G$1" pin="CTS"/>
@@
 <pinref part="JP1" gate="G$1" pin="GND"/>
 <label x="290.83" y="120.65" size="1.27" layer="95" xref="yes"/>
+</segment>
+<segment>
+<pinref part="PAD5" gate="1" pin="P"/>
+<wire x1="360.68" y1="35.56" x2="358.14" y2="35.56" width="0.1524" layer="91"/>
+<label x="358.14" y="35.56" size="1.778" layer="95" rot="R180" xref="yes"/>
+</segment>
+<segment>
+<pinref part="PAD4" gate="1" pin="P"/>
+<wire x1="360.68" y1="68.58" x2="358.14" y2="68.58" width="0.1524" layer="91"/>
+<label x="358.14" y="68.58" size="1.778" layer="95" rot="R180" xref="yes"/>
 </segment>
 </net>
@@
 <label x="290.83" y="110.49" size="1.27" layer="95" xref="yes"/>
 </segment>
+<segment>
+<pinref part="PAD1" gate="1" pin="P"/>
+<wire x1="360.68" y1="53.34" x2="358.14" y2="53.34" width="0.1524" layer="91"/>
+<label x="358.14" y="53.34" size="1.778" layer="95" rot="R180" xref="yes"/>
+</segment>
 </net>
 <net name="VCC" class="0">
@@
 <label x="290.83" y="115.57" size="1.27" layer="95" xref="yes"/>
 </segment>
-</net>
-<net name="RAW" class="1">
-<segment>
-<pinref part="PAD1" gate="1" pin="P"/>
-<wire x1="360.68" y1="66.04" x2="358.14" y2="66.04" width="0.1524" layer="91"/>
-<label x="358.14" y="66.04" size="1.778" layer="95" rot="R180" xref="yes"/>
+<segment>
+<pinref part="PAD3" gate="1" pin="P"/>
+<wire x1="360.68" y1="60.96" x2="358.14" y2="60.96" width="0.1524" layer="91"/>
+<label x="358.14" y="60.96" size="1.778" layer="95" rot="R180" xref="yes"/>
 </segment>
 </net>
@@
 <pinref part="JP1" gate="G$1" pin="TXO"/>
 <label x="290.83" y="113.03" size="1.27" layer="95" xref="yes"/>
+</segment>
+<segment>
+<pinref part="PAD2" gate="1" pin="P"/>
+<wire x1="360.68" y1="45.72" x2="358.14" y2="45.72" width="0.1524" layer="91"/>
+<label x="358.14" y="45.72" size="1.778" layer="95" rot="R180" xref="yes"/>
 </segment>
 </net>
@@
 </schematic>
 </drawing>
-<compatibility>
-<note version="8.2" severity="warning">
-Since Version 8.2, EAGLE supports online libraries. The ids
-of those online libraries will not be understood (or retained)
-with this version.
-</note>
-<note version="8.3" severity="warning">
-Since Version 8.3, EAGLE supports URNs for individual library
-assets (packages, symbols, and devices). The URNs of those assets
-will not be understood (or retained) with this version.
-</note>
-<note version="8.3" severity="warning">
-Since Version 8.3, EAGLE supports the association of 3D packages
-with devices in libraries, schematics, and board files. Those 3D
-packages will not be understood (or retained) with this version.
-</note>
-</compatibility>
 </eagle>

Commit message: Add files via upload
Parts:
- removed LED13: Green, Testing:LED
- removed R14: 330, SparkFun:RESISTOR0603-RES
- removed SJ3: SOLDERJUMPERNC, SparkFun-Passives:SOLDERJUMPERNC
- added H1, H2, H3: MOUNT-HOLE3.3, holes:MOUNT-HOLE3.3
Connections:
- removed net GND_SW: SJ3.2
- removed net N$11: LED13.A, R14.2
- removed net N$30: U$15.DOUT, U$16.DOUT
- removed net VDD: R11.2, R12.2, U$1.P$2, U$10.P$2, U$15.VDD, U$16.VDD, U$17.P$2, U$18.P$2, U$2.P$2, U$3.P$2, U$4.P$2, U$5.P$2, U$6.P$2, U$7.P$2, U$8.P$2, U$9.P$2
- net CLK: no longer R14.1
- net N$26: no longer SJ3.1
- net VCC: now also R11.2, R12.2, U$1.P$2, U$10.P$2, U$15.VDD, U$16.VDD, U$17.P$2, U$18.P$2, U$2.P$2, U$3.P$2, U$4.P$2, U$5.P$2, U$6.P$2, U$7.P$2, U$8.P$2, U$9.P$2
Other:
- moved on the sheet: C1, C2, C3, JP1, Q1, R11, R12, R13, R15, R16, S1, SJ2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

Commit message: Add files via upload
Parts:
- added C4, C5: (no value), resistor:C-USC0805K
- added IC1: MIC5219BM5, v-reg-micrel:MIC5219BM5
- added L1: (no value), rcl:L-USL2012C
- added SJ1, SJ3: SOLDERJUMPERNC, SparkFun-Passives:SOLDERJUMPERNC
- added SV1: (no value), con-lstb:MA04-2
- added U$19: DS3231_BACK, DS3231_BACK:DS3231_BACK
- added U$20: CR2032, CR2032:CR2032
- added U$21: USB-C, USB-C:USB-C
Connections:
- new net N$11: U$19.P$14, U$20.P$2
- new net N$29: SJ3.2, SV1.5
- new net N$30: SV1.3
- new net N$31: IC1.ADJ, L1.2
- new net RESET_WIFI: SJ1.1, SV1.6
- new net VCC_33: C4.1, IC1.OUT, L1.1, SV1.4, SV1.8
- net A4: now also U$19.P$15
- net A5: now also U$19.P$16
- net GND: now also C4.2, C5.2, IC1.GND, SJ1.2, SJ3.1, SV1.1, U$19.P$10, U$19.P$11, U$19.P$12, U$19.P$13, U$19.P$5, U$19.P$6, U$19.P$7, U$19.P$8, U$19.P$9, U$20.P$1, U$21.GND1, U$21.GND2, U$21.GND3, U$21.GND4, U$21.P$1, U$21.P$2, U$21.P$3, U$21.P$4
- net RXI: now also SV1.7
- net TXO: now also SV1.2
- net VCC: now also C5.1, IC1.EN, IC1.IN, U$19.P$2, U$21.VBUS1, U$21.VBUS2, U$21.VBUS3, U$21.VBUS4
Other:
- note added: "GND"
