File: Eagle/LocMap/LocationMapper.brd (EAGLE design)
At the start: 100 x 80 mm, 44 parts, among them Q1 8/16/20MHz, U1 ATMEGA328

Commit message: Add files via upload
Parts:
- added R17, R18: (no value), resistor:R0805
- added U$17, U$18: LED_LM, LED_LM:LED_LM
- moved LED13 263.3 mm to (60.5, 39.3)
- moved C1 233.4 mm to (101.2, 40.7)
- moved C2 233.4 mm to (107.5, 40.7)
- moved C3 233.4 mm to (63.1, 26.7)
- moved JP1 233.4 mm to (69.4, 15.3)
- moved Q1 233.4 mm to (87.2, 40.7)
- moved R13 233.4 mm to (69.4, 26.7)
- moved R14 233.4 mm to (75.8, 26.7)
- moved R15 233.4 mm to (82.1, 26.7)
- moved R16 233.4 mm to (88.5, 26.7)
- moved SJ2 233.4 mm to (92.3, 40.7)
- moved SJ3 233.4 mm to (96.1, 40.7)
- moved S1 233.4 mm to (79.6, 39.4)
- moved U1 220.9 mm to (84.3, 7.32), turned to 270 degrees
- moved U$13 208.6 mm to (150.4, 9.13)
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Connections:
- new net N$22: R18.1, U$18.P$1
- new net N$27: R17.1, U$17.P$1
- net GND: now also R17.2, R18.2
- net N$1: now also U$6.P$1; no longer U$1.P$2
- net N$10: now also U$5.P$1; no longer U$9.P$2
- net N$2: now also U$7.P$1; no longer U$2.P$2
- net N$3: now also U$8.P$1; no longer U$3.P$2
- net N$4: now also U$9.P$1; no longer U$4.P$2
- net N$5: now also U$10.P$1; no longer U$5.P$2
- net N$6: now also U$1.P$1; no longer U$10.P$2
- net N$7: now also U$2.P$1; no longer U$6.P$2
- net N$8: now also U$3.P$1; no longer U$7.P$2
- net N$9: now also U$4.P$1; no longer U$8.P$2
- net VDD: now also U$1.P$2, U$10.P$2, U$17.P$2, U$18.P$2, U$2.P$2, U$3.P$2, U$4.P$2, U$5.P$2, U$6.P$2, U$7.P$2, U$8.P$2, U$9.P$2; no longer U$1.P$1, U$10.P$1, U$2.P$1, U$3.P$1, U$4.P$1, U$5.P$1, U$6.P$1, U$7.P$1, U$8.P$1, U$9.P$1
Other:
- board size 100 x 80 mm -> 180 x 48.5 mm

Commit message: Add files via upload
Parts:
- added PAD3, PAD4, PAD5: (no value), wirepad:2,54/1,1
- moved U$10 102.3 mm to (115.0, 39.0)
- moved C2 97.5 mm to (10.5, 30.5), turned to 180 degrees
- moved SJ3 78.4 mm to (20.5, 20.1)
- moved U$9 77.5 mm to (95.0, 39.0)
- moved SJ2 74.0 mm to (20.5, 22.7)
- moved JP1 67.3 mm to (3.82, 30.5), turned to 270 degrees
- moved S1 66.6 mm to (14.7, 24.5)
- moved U$1 65.0 mm to (115.0, 9.50)
- moved R4 56.4 mm to (82.1, 33.7), turned to 180 degrees
- moved R13 54.5 mm to (15.0, 30.5)
- moved U$8 52.8 mm to (75.0, 39.0)
- moved U$2 51.6 mm to (95.0, 9.50)
- moved C1 43.0 mm to (64.2, 18.7), turned to 180 degrees
- moved Q1 42.2 mm to (47.1, 27.7), turned to 225 degrees
- moved R3 42.0 mm to (72.0, 31.9)
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Connections:
- removed net RAW: PAD1.1
- net GND: now also PAD4.1, PAD5.1; no longer PAD2.1
- net RXI: now also PAD2.1
- net TXO: now also PAD1.1
- net VCC: now also PAD3.1
Routing:
- net VDD: track 0.00 -> 245.1 mm
- net N$6: track 0.00 -> 70.0 mm
- net SEGE2: track 0.00 -> 51.3 mm, vias 0 -> 1
- net SEGDP2: track 0.00 -> 50.1 mm, vias 0 -> 1
- net SEGD2: track 0.00 -> 49.8 mm, vias 0 -> 1
- net DIG32: track 0.00 -> 49.0 mm
- net N$7: track 0.00 -> 49.0 mm
- net SEGC2: track 0.00 -> 48.6 mm, vias 0 -> 1
- net SEGG2: track 0.00 -> 46.6 mm, vias 0 -> 1
- net DIG22: track 0.00 -> 46.2 mm
- net SEGB2: track 0.00 -> 45.9 mm
- net DIG12: track 0.00 -> 38.3 mm
- net N$1: track 0.00 -> 38.2 mm
- net DIG02: track 0.00 -> 37.6 mm
- net SEGF2: track 0.00 -> 35.6 mm
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- added copper zone on layer 1, net GND

Commit message: Add files via upload
Parts:
- removed LED13: Green, Testing:0603-LED-ALT1
- removed R14: 330, SparkFun:0603-RES
- removed SJ3: (no value), SparkFun-Passives:SJ_2S
- added H1, H2, H3: MOUNT-HOLE3.3, holes:3,3
- moved R18 13.9 mm to (14.5, 19.6), turned to 0 degrees
- moved R17 12.4 mm to (14.5, 31.3), turned to 0 degrees
- moved R13 5.73 mm to (20.5, 28.9)
- moved C2 4.27 mm to (14.5, 29.0)
- moved C1 3.98 mm to (60.3, 19.5)
- moved SJ2 2.01 mm to (19.8, 24.6), turned to 90 degrees
- moved R15 1.12 mm to (61.8, 29.7)
- moved R12 1.10 mm to (117.2, 31.9)
- moved R16 0.92 mm to (59.6, 29.7)
- moved R11 0.81 mm to (94.9, 31.7)
- moved C3 0.70 mm to (50.8, 29.6)
Connections:
- removed net GND_SW: SJ3.2
- removed net N$11: LED13.A, R14.2
- removed net N$30: U$15.P$1, U$16.P$1
- removed net VDD: R11.2, R12.2, U$1.P$2, U$10.P$2, U$15.P$16, U$16.P$16, U$17.P$2, U$18.P$2, U$2.P$2, U$3.P$2, U$4.P$2, U$5.P$2, U$6.P$2, U$7.P$2, U$8.P$2, U$9.P$2
- net CLK: no longer R14.1
- net N$26: no longer SJ3.1
- net VCC: now also R11.2, R12.2, U$1.P$2, U$10.P$2, U$15.P$16, U$16.P$16, U$17.P$2, U$18.P$2, U$2.P$2, U$3.P$2, U$4.P$2, U$5.P$2, U$6.P$2, U$7.P$2, U$8.P$2, U$9.P$2
Routing:
- net VCC: track 28.3 -> 443.8 mm, vias 0 -> 13
- net VDD: track 245.1 -> 0.00 mm
- net DIG21: track 0.00 -> 107.0 mm, vias 0 -> 2
- net RXI: track 4.38 -> 104.4 mm
- net DIG01: track 0.00 -> 93.0 mm, vias 0 -> 3
- net TXO: track 4.13 -> 96.5 mm, vias 1 -> 2
- net CLK: track 0.00 -> 81.5 mm, vias 0 -> 2
- net LCSN2: track 0.00 -> 75.5 mm, vias 0 -> 2
- net DIN2: track 0.00 -> 72.3 mm
- net DIG31: track 0.00 -> 67.4 mm, vias 0 -> 1
- net DIG11: track 0.00 -> 65.9 mm, vias 0 -> 1
- net SEGB1: track 0.00 -> 65.4 mm, vias 0 -> 1
- net SEGDP1: track 0.00 -> 63.9 mm, vias 0 -> 1
- net LCSN1: track 0.00 -> 63.2 mm, vias 0 -> 2
- net SEGG1: track 0.00 -> 63.1 mm, vias 0 -> 1
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- added copper zone on layer 16, net GND

Commit message: Add files via upload
Routing:
- net VCC: track 443.8 -> 451.4 mm
Changed lines of the file:
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@@
 <wire x1="96.4" y1="35.5" x2="99" y2="38.1" width="0.6096" layer="16"/>
 <wire x1="94.1" y1="35.5" x2="94.1" y2="33.8" width="0.6096" layer="1"/>
-<wire x1="94.1" y1="33.8" x2="94.1" y2="31.59" width="0.6096" layer="1"/>
+<wire x1="94.1" y1="33.8" x2="94.1" y2="31.9" width="0.6096" layer="1"/>
+<wire x1="94.1" y1="31.9" x2="94.1" y2="31.59" width="0.6096" layer="1"/>
 <wire x1="94.1" y1="31.59" x2="94.145" y2="31.545" width="0.6096" layer="1"/>
 <wire x1="99" y1="38.1" x2="99" y2="39.2" width="0.6096" layer="16"/>
@@
 <wire x1="116.22" y1="31.85" x2="115.526953125" y2="32.07599375" width="0.4064" layer="1"/>
 <wire x1="115.526953125" y1="32.07599375" x2="115.3" y2="32.15" width="0.4064" layer="1"/>
-<wire x1="115.3" y1="32.15" x2="115.735" y2="31.715" width="0.4064" layer="1"/>
+<wire x1="115.3" y1="32.15" x2="115.525" y2="31.925" width="0.4064" layer="1"/>
+<wire x1="115.525" y1="31.925" x2="115.735" y2="31.715" width="0.4064" layer="1"/>
 <wire x1="115.735" y1="31.715" x2="115.885" y2="31.715" width="0.4064" layer="1"/>
 <wire x1="116.22" y1="31.85" x2="115.735" y2="31.565" width="0.4064" layer="1"/>
@@
 <wire x1="115" y1="31.8" x2="115.3" y2="31.8" width="0.4064" layer="1"/>
 <via x="117.7" y="36.7" extent="1-16" drill="0.6"/>
-<wire x1="114.6" y1="32.2" x2="117.7" y2="35.3" width="0.4064" layer="16"/>
-<wire x1="117.7" y1="35.3" x2="117.7" y2="36.7" width="0.4064" layer="16"/>
-<wire x1="117.7" y1="36.7" x2="117.7" y2="37.697" width="0.4064" layer="1"/>
-<wire x1="117.7" y1="37.697" x2="116.397" y2="39" width="0.4064" layer="1"/>
 <via x="60.7" y="32" extent="1-16" drill="0.6"/>
 <wire x1="60.7" y1="32" x2="60.7" y2="30.57" width="0.4064" layer="1"/>
@@
 <wire x1="114.6" y1="32.2" x2="114.72400625" y2="32.07599375" width="0.6096" layer="1"/>
 <wire x1="114.72400625" y1="32.07599375" x2="115.526953125" y2="32.07599375" width="0.6096" layer="1"/>
+<wire x1="94.33" y1="28.2" x2="94.33" y2="31.67" width="0.6096" layer="1"/>
+<wire x1="94.33" y1="31.67" x2="94.1" y2="31.9" width="0.6096" layer="1"/>
+<wire x1="115.4" y1="28.19" x2="115.4" y2="31.8" width="0.6096" layer="1"/>
+<wire x1="115.4" y1="31.8" x2="115.525" y2="31.925" width="0.6096" layer="1"/>
+<wire x1="117.7" y1="36.7" x2="117.7" y2="37.697" width="0.6096" layer="1"/>
+<wire x1="117.7" y1="37.697" x2="116.397" y2="39" width="0.6096" layer="1"/>
+<wire x1="114.6" y1="32.2" x2="117.7" y2="35.3" width="0.6096" layer="16"/>
+<wire x1="117.7" y1="35.3" x2="117.7" y2="36.7" width="0.6096" layer="16"/>
 </signal>
 <signal name="A4">

Commit message: Add files via upload
Parts:
- added C4, C5: (no value), resistor:C0805K
- added IC1: MIC5219BM5, v-reg-micrel:SOT23-5
- added L1: (no value), rcl:L2012C
- added SJ1, SJ3: (no value), SparkFun-Passives:SJ_2S
- added SV1: (no value), con-lstb:MA04-2
- added U$19: DS3231_BACK, DS3231_BACK:DS3231_BACK
- added U$20: CR2032, CR2032:CR2032
- added U$21: USB-C, USB-C:USB-C
- moved R5 6.36 mm to (85.3, 36.9)
- moved R4 6.19 mm to (85.3, 39.0)
- moved R1 3.51 mm to (66.6, 32.9)
- moved R2 3.01 mm to (66.6, 34.9)
Connections:
- new net N$11: U$19.P$14, U$20.P$2, U$20.P$3
- new net N$29: SJ3.2, SV1.5
- new net N$30: SV1.3
- new net N$31: IC1.4, L1.2
- new net RESET_WIFI: SJ1.1, SV1.6
- new net VCC_33: C4.1, IC1.5, L1.1, SV1.4, SV1.8
- net A4: now also U$19.P$15
- net A5: now also U$19.P$16
- net GND: now also C4.2, C5.2, IC1.2, SJ1.2, SJ3.1, SV1.1, U$19.P$10, U$19.P$11, U$19.P$12, U$19.P$13, U$19.P$5, U$19.P$6, U$19.P$7, U$19.P$8, U$19.P$9, U$20.P$1, U$21.GND, U$21.GND1, U$21.GND2, U$21.GND3, U$21.P$10, U$21.P$7, U$21.P$8, U$21.P$91
- net RXI: now also SV1.7
- net TXO: now also SV1.2
- net VCC: now also C5.1, IC1.1, IC1.3, U$19.P$2, U$21.VBUS1, U$21.VBUS2, U$21.VBUS3, U$21.VBUS4
Routing:
- net GND: track 28.4 -> 132.5 mm, vias 18 -> 25
- net N$11: track 0.00 -> 78.1 mm
- net VCC: track 451.4 -> 518.2 mm, vias 13 -> 17
- net VCC_33: track 0.00 -> 24.8 mm
- net TXO: track 96.5 -> 119.9 mm, vias 2 -> 3
- net RXI: track 104.4 -> 120.4 mm
- net A4: track 3.95 -> 18.2 mm, vias 0 -> 1
- net A5: track 2.92 -> 15.5 mm, vias 0 -> 1
- net N$29: track 0.00 -> 8.87 mm
- net RESET_WIFI: track 0.00 -> 7.57 mm
- net N$16: track 7.85 -> 13.3 mm
- net N$5: track 33.8 -> 28.3 mm
- net N$4: track 12.8 -> 7.40 mm
- net N$15: track 10.4 -> 15.8 mm
- net LED5S: track 40.6 -> 45.1 mm
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
Commit message: Add files via upload
Parts:
- moved R17 0.80 mm to (14.5, 32.1)
Routing:
- net N$27: track 7.79 -> 6.99 mm
Other:
- board text added: "*"
- board text added: "10uF"
- board text added: "1uH"
- board text added: "22uF"
- board text added: "5V"
- board text added: "BLK"
- board text added: "GND"
- board text added: "GRN"
- board text added: "RX"
- board text added: "TX"
